File: hardware/pcb-a/pcb-a.kicad_pcb (KiCad board)
At the start: 2 copper layers, 110 x 120 mm, 29 parts, among them J1 ESP32 socket left row, J2 ESP32 socket right row, J3 PH sensor, J4 DO sensor, J5 TURB sensor, J6 CO2 sensor, J7 DS18B20, J8 I2C expansion, J9 PCB-B relay connector, U1 ADS1115

Commit message: Fix KiCad circuit values and placements
Co-authored-by: tomnyle <175001228+tomnyle@users.noreply.github.com>
Parts:
- added J10: DHT22, SmartFarm:SF_PinHeader_1x3, F.Cu at (15.0, 115.0)
- added R13: 4.7k pull-up, SmartFarm:SF_R_0603, F.Cu at (22.0, 115.0)
- moved C2 16.3 mm to (82.0, 84.0)
- moved C1 7.07 mm to (72.0, 84.0)
Connections:
- J1 pad 3: (no net) -> DHT22_DATA

Commit message: Align PCB documentation with KiCad projects
Co-authored-by: tomnyle <175001228+tomnyle@users.noreply.github.com>
Parts:
- R1, R3, R5, R7: value 10k -> 12k
