File: hardware/pcb-a/pcb-a.kicad_sch (KiCad schematic)
At the start: 29 parts, among them J1 ESP32 DevKit 30-pin socket row, J2 ESP32 DevKit 30-pin socket row, J3 PH sensor, J4 DO sensor, J5 TURB sensor, J6 CO2 sensor, J7 DS18B20, J8 I2C expansion (BH1750), J9 PCB-B relay interface, U1 ADS1115 (ADDR=GND)

Commit message: Fix KiCad circuit values and placements
Co-authored-by: tomnyle <175001228+tomnyle@users.noreply.github.com>
Parts:
- added J10: DHT22, SmartFarm:SF_PinHeader_1x3, symbol SmartFarm:Conn_01x03
- added R13: 4.7k, SmartFarm:SF_R_0603, symbol SmartFarm:R
- R1, R3, R5, R7: value 10k 1% -> 12k 1%
Connections:
- net 3V3: now also J10.1, R13.1
- net GND: now also J10.3
- net GPIO15 renamed DHT22_DATA
- net DHT22_DATA: now also J10.2, R13.2
- no-connect marks 0 -> 1
