File: hardware/pcb-b/pcb-b.kicad_pcb (KiCad board)
At the start: 2 copper layers, 95 x 65 mm, 43 parts, among them J1 PCB-A J_AB, J2 Relay module input 1-4, J3 Relay module input 5-8, Q1 BC817-40, Q2 BC817-40, Q3 BC817-40, Q4 BC817-40, Q5 BC817-40, Q6 BC817-40, Q7 BC817-40, Q8 BC817-40

Commit message: Fix KiCad circuit values and placements
Co-authored-by: tomnyle <175001228+tomnyle@users.noreply.github.com>
Parts:
- R1, R2, R3, R4, R5, R6, R7, R8: value 4.7k base -> 2.2k base
