File: hardware/pcb-b/pcb-b.kicad_sch (KiCad schematic)
At the start: 43 parts, among them J1 Mates to PCB-A J_AB, J2 Relay module inputs 1-4, J3 Relay module inputs 5-8, Q1 BC817-40 low-side sink, Q2 BC817-40 low-side sink, Q3 BC817-40 low-side sink, Q4 BC817-40 low-side sink, Q5 BC817-40 low-side sink, Q6 BC817-40 low-side sink, Q7 BC817-40 low-side sink, Q8 BC817-40 low-side sink

Commit message: Fix KiCad circuit values and placements
Co-authored-by: tomnyle <175001228+tomnyle@users.noreply.github.com>
Parts:
- R1, R2, R3, R4, R5, R6, R7, R8: value 4.7k base -> 2.2k base
Changed lines of the file:
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@@
 		(instances
 			(project "SmartFarm PCB-B Relay Interface"
-				(path "/859089c3-6b32-43d2-acd7-2e64ce11fe46"
+				(path "/c2a9b746-bc05-4c2a-a3f0-01e3628a7244"
 					(reference "J1")
 					(unit 1)
@@
 			)
 		)
-		(property "Value" "4.7k base"
+		(property "Value" "2.2k base"
 			(at 64.77 44.45 0.0000)
 			(effects
@@
 		(instances
 			(project "SmartFarm PCB-B Relay Interface"
-				(path "/859089c3-6b32-43d2-acd7-2e64ce11fe46"
+				(path "/c2a9b746-bc05-4c2a-a3f0-01e3628a7244"
 					(reference "R1")
 					(unit 1)
@@
 		(instances
 			(project "SmartFarm PCB-B Relay Interface"
-				(path "/859089c3-6b32-43d2-acd7-2e64ce11fe46"
+				(path "/c2a9b746-bc05-4c2a-a3f0-01e3628a7244"
 					(reference "Q1")
 					(unit 1)
@@
 		(instances
 			(project "SmartFarm PCB-B Relay Interface"
-				(path "/859089c3-6b32-43d2-acd7-2e64ce11fe46"
+				(path "/c2a9b746-bc05-4c2a-a3f0-01e3628a7244"
 					(reference "R9")
 					(unit 1)
@@
 		(instances
 			(project "SmartFarm PCB-B Relay Interface"
-				(path "/859089c3-6b32-43d2-acd7-2e64ce11fe46"
+				(path "/c2a9b746-bc05-4c2a-a3f0-01e3628a7244"
 					(reference "R17")
 					(unit 1)
@@
 		(instances
 			(project "SmartFarm PCB-B Relay Interface"
-				(path "/859089c3-6b32-43d2-acd7-2e64ce11fe46"
+				(path "/c2a9b746-bc05-4c2a-a3f0-01e3628a7244"
 					(reference "D1")
 					(unit 1)
@@
 			)
 		)
-		(property "Value" "4.7k base"
+		(property "Value" "2.2k base"
 			(at 64.77 64.77 0.0000)
 			(effects
@@
 		(instances
 			(project "SmartFarm PCB-B Relay Interface"
-				(path "/859089c3-6b32-43d2-acd7-2e64ce11fe46"
+				(path "/c2a9b746-bc05-4c2a-a3f0-01e3628a7244"
 					(reference "R2")
 					(unit 1)
@@
 		(instances
 			(project "SmartFarm PCB-B Relay Interface"
-				(path "/859089c3-6b32-43d2-acd7-2e64ce11fe46"
+				(path "/c2a9b746-bc05-4c2a-a3f0-01e3628a7244"
 					(reference "Q2")
 					(unit 1)
@@
 		(instances
 			(project "SmartFarm PCB-B Relay Interface"
-				(path "/859089c3-6b32-43d2-acd7-2e64ce11fe46"
+				(path "/c2a9b746-bc05-4c2a-a3f0-01e3628a7244"
 					(reference "R10")
 					(unit 1)
@@
 		(instances
 			(project "SmartFarm PCB-B Relay Interface"
-				(path "/859089c3-6b32-43d2-acd7-2e64ce11fe46"
+				(path "/c2a9b746-bc05-4c2a-a3f0-01e3628a7244"
 					(reference "R18")
 					(unit 1)
@@
 		(instances
 			(project "SmartFarm PCB-B Relay Interface"
-				(path "/859089c3-6b32-43d2-acd7-2e64ce11fe46"
+				(path "/c2a9b746-bc05-4c2a-a3f0-01e3628a7244"
 					(reference "D2")
 					(unit 1)
@@
 			)
 		)
-		(property "Value" "4.7k base"
+		(property "Value" "2.2k base"
 			(at 64.77 85.09 0.0000)
 			(effects
@@
 		(instances
 			(project "SmartFarm PCB-B Relay Interface"
-				(path "/859089c3-6b32-43d2-acd7-2e64ce11fe46"
+				(path "/c2a9b746-bc05-4c2a-a3f0-01e3628a7244"
 					(reference "R3")
 					(unit 1)
@@
 		(instances
 			(project "SmartFarm PCB-B Relay Interface"
-				(path "/859089c3-6b32-43d2-acd7-2e64ce11fe46"
+				(path "/c2a9b746-bc05-4c2a-a3f0-01e3628a7244"
 					(reference "Q3")
 					(unit 1)
@@
 		(instances
 			(project "SmartFarm PCB-B Relay Interface"
-				(path "/859089c3-6b32-43d2-acd7-2e64ce11fe46"
+				(path "/c2a9b746-bc05-4c2a-a3f0-01e3628a7244"
 					(reference "R11")
 					(unit 1)
@@
 		(instances
 			(project "SmartFarm PCB-B Relay Interface"
-				(path "/859089c3-6b32-43d2-acd7-2e64ce11fe46"
+				(path "/c2a9b746-bc05-4c2a-a3f0-01e3628a7244"
 					(reference "R19")
 					(unit 1)
@@
 		(instances
 			(project "SmartFarm PCB-B Relay Interface"
-				(path "/859089c3-6b32-43d2-acd7-2e64ce11fe46"
+				(path "/c2a9b746-bc05-4c2a-a3f0-01e3628a7244"
 					(reference "D3")
 					(unit 1)
@@
 			)
 		)
-		(property "Value" "4.7k base"
+		(property "Value" "2.2k base"
 			(at 64.77 105.41 0.0000)
 			(effects
@@
 		(instances
 			(project "SmartFarm PCB-B Relay Interface"
-				(path "/859089c3-6b32-43d2-acd7-2e64ce11fe46"
+				(path "/c2a9b746-bc05-4c2a-a3f0-01e3628a7244"
 					(reference "R4")
 					(unit 1)
@@
 		(instances
 			(project "SmartFarm PCB-B Relay Interface"
-				(path "/859089c3-6b32-43d2-acd7-2e64ce11fe46"
+				(path "/c2a9b746-bc05-4c2a-a3f0-01e3628a7244"
 					(reference "Q4")
 					(unit 1)
@@
 		(instances
 			(project "SmartFarm PCB-B Relay Interface"
-				(path "/859089c3-6b32-43d2-acd7-2e64ce11fe46"
+				(path "/c2a9b746-bc05-4c2a-a3f0-01e3628a7244"
 					(reference "R12")
 					(unit 1)
@@
 		(instances
 			(project "SmartFarm PCB-B Relay Interface"
-				(path "/859089c3-6b32-43d2-acd7-2e64ce11fe46"
+				(path "/c2a9b746-bc05-4c2a-a3f0-01e3628a7244"
 					(reference "R20")
 					(unit 1)
@@
 		(instances
 			(project "SmartFarm PCB-B Relay Interface"
-				(path "/859089c3-6b32-43d2-acd7-2e64ce11fe46"
+				(path "/c2a9b746-bc05-4c2a-a3f0-01e3628a7244"
 					(reference "D4")
 					(unit 1)
@@
 			)
 		)
-		(property "Value" "4.7k base"
+		(property "Value" "2.2k base"
 			(at 64.77 124.46 0.0000)
 			(effects
@@
 		(instances
 			(project "SmartFarm PCB-B Relay Interface"
-				(path "/859089c3-6b32-43d2-acd7-2e64ce11fe46"
+				(path "/c2a9b746-bc05-4c2a-a3f0-01e3628a7244"
 					(reference "R5")
 					(unit 1)
@@
 		(instances
 			(project "SmartFarm PCB-B Relay Interface"
-				(path "/859089c3-6b32-43d2-acd7-2e64ce11fe46"
+				(path "/c2a9b746-bc05-4c2a-a3f0-01e3628a7244"
 					(reference "Q5")
 					(unit 1)
@@
 		(instances
 			(project "SmartFarm PCB-B Relay Interface"
-				(path "/859089c3-6b32-43d2-acd7-2e64ce11fe46"
+				(path "/c2a9b746-bc05-4c2a-a3f0-01e3628a7244"
 					(reference "R13")
 					(unit 1)
@@
 		(instances
 			(project "SmartFarm PCB-B Relay Interface"
-				(path "/859089c3-6b32-43d2-acd7-2e64ce11fe46"
+				(path "/c2a9b746-bc05-4c2a-a3f0-01e3628a7244"
 					(reference "R21")
 					(unit 1)
@@
 		(instances
 			(project "SmartFarm PCB-B Relay Interface"
-				(path "/859089c3-6b32-43d2-acd7-2e64ce11fe46"
+				(path "/c2a9b746-bc05-4c2a-a3f0-01e3628a7244"
 					(reference "D5")
 					(unit 1)
@@
 			)
 		)
-		(property "Value" "4.7k base"
+		(property "Value" "2.2k base"
 			(at 64.77 144.78 0.0000)
 			(effects
@@
 		(instances
 			(project "SmartFarm PCB-B Relay Interface"
-				(path "/859089c3-6b32-43d2-acd7-2e64ce11fe46"
+				(path "/c2a9b746-bc05-4c2a-a3f0-01e3628a7244"
 					(reference "R6")
 					(unit 1)
@@
 		(instances
 			(project "SmartFarm PCB-B Relay Interface"
-				(path "/859089c3-6b32-43d2-acd7-2e64ce11fe46"
+				(path "/c2a9b746-bc05-4c2a-a3f0-01e3628a7244"
 					(reference "Q6")
 					(unit 1)
@@
 		(instances
 			(project "SmartFarm PCB-B Relay Interface"
-				(path "/859089c3-6b32-43d2-acd7-2e64ce11fe46"
+				(path "/c2a9b746-bc05-4c2a-a3f0-01e3628a7244"
 					(reference "R14")
 					(unit 1)
@@
 		(instances
 			(project "SmartFarm PCB-B Relay Interface"
-				(path "/859089c3-6b32-43d2-acd7-2e64ce11fe46"
+				(path "/c2a9b746-bc05-4c2a-a3f0-01e3628a7244"
 					(reference "R22")
 					(unit 1)
@@
 		(instances
 			(project "SmartFarm PCB-B Relay Interface"
-				(path "/859089c3-6b32-43d2-acd7-2e64ce11fe46"
+				(path "/c2a9b746-bc05-4c2a-a3f0-01e3628a7244"
 					(reference "D6")
 					(unit 1)
@@
 			)
 		)
-		(property "Value" "4.7k base"
+		(property "Value" "2.2k base"
 			(at 64.77 165.1 0.0000)
 			(effects
@@
 		(instances
 			(project "SmartFarm PCB-B Relay Interface"
-				(path "/859089c3-6b32-43d2-acd7-2e64ce11fe46"
+				(path "/c2a9b746-bc05-4c2a-a3f0-01e3628a7244"
 					(reference "R7")
 					(unit 1)
@@
 		(instances
 			(project "SmartFarm PCB-B Relay Interface"
-				(path "/859089c3-6b32-43d2-acd7-2e64ce11fe46"
+				(path "/c2a9b746-bc05-4c2a-a3f0-01e3628a7244"
 					(reference "Q7")
 					(unit 1)
@@
 		(instances
 			(project "SmartFarm PCB-B Relay Interface"
-				(path "/859089c3-6b32-43d2-acd7-2e64ce11fe46"
+				(path "/c2a9b746-bc05-4c2a-a3f0-01e3628a7244"
 					(reference "R15")
 					(unit 1)
@@
 		(instances
 			(project "SmartFarm PCB-B Relay Interface"
-				(path "/859089c3-6b32-43d2-acd7-2e64ce11fe46"
+				(path "/c2a9b746-bc05-4c2a-a3f0-01e3628a7244"
 					(reference "R23")
 					(unit 1)
@@
 		(instances
 			(project "SmartFarm PCB-B Relay Interface"
-				(path "/859089c3-6b32-43d2-acd7-2e64ce11fe46"
+				(path "/c2a9b746-bc05-4c2a-a3f0-01e3628a7244"
 					(reference "D7")
 					(unit 1)
@@
 			)
 		)
-		(property "Value" "4.7k base"
+		(property "Value" "2.2k base"
 			(at 64.77 185.42 0.0000)
 			(effects
@@
 		(instances
 			(project "SmartFarm PCB-B Relay Interface"
-				(path "/859089c3-6b32-43d2-acd7-2e64ce11fe46"
+				(path "/c2a9b746-bc05-4c2a-a3f0-01e3628a7244"
 					(reference "R8")
 					(unit 1)
@@
 		(instances
 			(project "SmartFarm PCB-B Relay Interface"
-				(path "/859089c3-6b32-43d2-acd7-2e64ce11fe46"
+				(path "/c2a9b746-bc05-4c2a-a3f0-01e3628a7244"
 					(reference "Q8")
 					(unit 1)
@@
 		(instances
 			(project "SmartFarm PCB-B Relay Interface"
-				(path "/859089c3-6b32-43d2-acd7-2e64ce11fe46"
+				(path "/c2a9b746-bc05-4c2a-a3f0-01e3628a7244"
 					(reference "R16")
 					(unit 1)
@@
 		(instances
 			(project "SmartFarm PCB-B Relay Interface"
-				(path "/859089c3-6b32-43d2-acd7-2e64ce11fe46"
+				(path "/c2a9b746-bc05-4c2a-a3f0-01e3628a7244"
 					(reference "R24")
 					(unit 1)
@@
 		(instances
 			(project "SmartFarm PCB-B Relay Interface"
-				(path "/859089c3-6b32-43d2-acd7-2e64ce11fe46"
+				(path "/c2a9b746-bc05-4c2a-a3f0-01e3628a7244"
 					(reference "D8")
 					(unit 1)
@@
 		(instances
 			(project "SmartFarm PCB-B Relay Interface"
-				(path "/859089c3-6b32-43d2-acd7-2e64ce11fe46"
+				(path "/c2a9b746-bc05-4c2a-a3f0-01e3628a7244"
 					(reference "J2")
 					(unit 1)
@@
 		(instances
 			(project "SmartFarm PCB-B Relay Interface"
-				(path "/859089c3-6b32-43d2-acd7-2e64ce11fe46"
+				(path "/c2a9b746-bc05-4c2a-a3f0-01e3628a7244"
 					(reference "J3")
 					(unit 1)
